File: standalone/ospreys/ospreys.kicad_sch (KiCad schematic)
At the start: 59 parts, among them J1 USB_B, J10 AudioJack2_SwitchT, J11 AudioJack2_SwitchT, J13 Conn_02x02_Odd_Even, J15 Conn_02x02_Odd_Even, J16 Conn_02x02_Odd_Even, J17 Conn_02x02_Odd_Even, J18 Conn_02x02_Odd_Even, J19 Conn_02x02_Odd_Even, J20 Conn_02x02_Odd_Even, J22 Conn_02x03_Odd_Even, J23 Conn_02x03_Odd_Even, J24 Conn_02x03_Odd_Even, J25 Conn_02x03_Odd_Even, J26 Conn_02x03_Odd_Even, J27 Conn_02x03_Odd_Even, J28 Conn_02x03_Odd_Even, J29 Conn_02x02_Odd_Even, J31 Conn_02x02_Odd_Even, J32 Conn_02x02_Odd_Even, J33 Conn_02x02_Odd_Even, J34 Conn_02x02_Odd_Even, J35 Conn_02x02_Odd_Even, J36 Conn_02x02_Odd_Even, J37 Conn_02x02_Odd_Even, J38 Conn_02x02_Odd_Even, J39 Conn_02x02_Odd_Even, J40 Conn_02x02_Odd_Even, J41 Conn_02x02_Odd_Even, J5 AudioJack2_SwitchT, J6 AudioJack2_SwitchT, J7 AudioJack2_SwitchT, J8 AudioJack2_SwitchT, J9 AudioJack2_SwitchT

Commit message: more
Parts:
- removed J2: (no value), symbol Connector:Conn_01x03_Male
- removed J3: (no value), symbol Connector:Conn_01x03_Female
- added H1: (no value), symbol Mechanical:MountingHole
- added H10, H11, H12, H7, H8, H9: MountingHole, MountingHole:MountingHole_3.2mm_M3, symbol Mechanical:MountingHole
- added H13, H14, H15, H16, H17, H18, H19, H2, H20, H21, H22, H23, H24, H25, H26, H27, H28, H29, H3, H4, H5, H6: MountingHole, symbol Mechanical:MountingHole
- added J2: Conn_02x03_Odd_Even, Connector_PinSocket_2.54mm:PinSocket_2x03_P2.54mm_Vertical_SMD, symbol Connector_Generic:Conn_02x03_Odd_Even
- added J3: (no value), symbol Connector_Generic:Conn_02x03_Odd_Even
- added R3: (no value), Resistor_SMD:R_0805_2012Metric_Pad1.20x1.40mm_HandSolder, symbol Device:R
- added R4, R5, R6: 10k, Resistor_SMD:R_0805_2012Metric_Pad1.20x1.40mm_HandSolder, symbol Device:R
- J1: value USB_B -> (none); footprint Connector_USB:USB_B_Lumberg_2411_02_Horizontal -> (none)
- J31, J33, J34, J35, J36, J37, J38, J39, J40, J41: footprint (none) -> Connector_PinHeader_2.54mm:PinHeader_2x02_P2.54mm_Vertical_SMD
- renumbered J14 to J13, J13 to J14, J29 to J21, J21 to J22, J22 to J23, J23 to J24, J24 to J25, J25 to J26, J26 to J27, J27 to J28, J28 to J29
Connections:
- net +12V: now also J2.1 (Pin_1), J2.2 (Pin_2)
- net +12VA: now also J30.4 (Pin_4), J31.4 (Pin_4), J34.4 (Pin_4), J35.4 (Pin_4), J38.4 (Pin_4), J39.4 (Pin_4), J3.1 (Pin_1), J3.2 (Pin_2); no longer J30.1 (Pin_1), J31.1 (Pin_1), J34.1 (Pin_1), J35.1 (Pin_1), J38.1 (Pin_1), J39.1 (Pin_1)
- net -12V: now also J2.5 (Pin_5), J2.6 (Pin_6)
- net -12VA: now also J32.1 (Pin_1), J33.1 (Pin_1), J36.1 (Pin_1), J37.1 (Pin_1), J40.1 (Pin_1), J41.1 (Pin_1), J3.5 (Pin_5), J3.6 (Pin_6); no longer J32.4 (Pin_4), J33.4 (Pin_4), J36.4 (Pin_4), J37.4 (Pin_4), J40.4 (Pin_4), J41.4 (Pin_4)
- net GND: now also J2.3 (Pin_3), J2.4 (Pin_4)
- net GND1: now also J30.1 (Pin_1), J31.1 (Pin_1), J32.4 (Pin_4), J33.4 (Pin_4), J34.1 (Pin_1), J35.1 (Pin_1), J36.4 (Pin_4), J37.4 (Pin_4), J38.1 (Pin_1), J39.1 (Pin_1), J40.4 (Pin_4), J41.4 (Pin_4), J3.3 (Pin_3), J3.4 (Pin_4); no longer J30.4 (Pin_4), J31.4 (Pin_4), J32.1 (Pin_1), J33.1 (Pin_1), J34.4 (Pin_4), J35.4 (Pin_4), J36.1 (Pin_1), J37.1 (Pin_1), J38.4 (Pin_4), J39.4 (Pin_4), J40.1 (Pin_1), J41.1 (Pin_1)
- net at J14.1 (Pin_1), J5.T: no longer J14.2 (Pin_2)
- net at J14.3 (Pin_3), J5.TN: no longer J14.4 (Pin_4)
- new net: R3.1, R5.1, RV1.3
- new net: R4.2, R6.2, RV1.6
- new net: J21.1 (Pin_1), R4.1
- new net: J21.2 (Pin_2), R6.1
- new net: J21.3 (Pin_3), R3.2
- new net: J21.4 (Pin_4), R5.2
Other:
- moved on the sheet: J10, J11, J12, J13, J14, J15, J16, J17, J18, J19, J20, J21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
