File: eurorack/accessories/chordata/chordata.kicad_pcb (KiCad board)
At the start: 2 copper layers, 20.3 x 45.7 mm, 44 parts, among them J1 USB_C_Receptacle_USB2.0, J2 Conn_02x05_Odd_Even, J3 Conn_01x18, J4 Conn_01x18, SW1 SW_Push, SW2 SW_Push, U1 MIC5219-3.3YM5, U2 RP2040, U3 W25Q128JVS, Y1 Crystal_GND24

Commit message: final chordata v1 layout
Parts:
- added H1: MountingHole, Pale Slim Ghost:hole JLCPCB tooling, F.Cu at (108.5, 34.3)
- added H2: MountingHole, Pale Slim Ghost:hole JLCPCB tooling, F.Cu at (94.6, 76.2)
- D3: footprint LED_SMD:LED_0402_1005Metric -> LED_SMD:LED_0603_1608Metric
- R3, R5: value 27 -> 22
- SW1, SW2: footprint Pale Slim Ghost:SW_Push_1P1T_NO_CK_KMR2 -> Pale Slim Ghost:SW_Push_1P1T_SKSGACE010
- moved D3 0.51 mm to (108.0, 41.8)
Connections:
- J1 pad A6: /USB_D- -> /USB_D+
- J1 pad A7: /USB_D+ -> /USB_D-
- J1 pad B6: /USB_D- -> /USB_D+
- J1 pad B7: /USB_D+ -> /USB_D-
Routing:
- net GND: track 57.4 -> 52.7 mm, vias 11 -> 12
- net /USB_D-: track 13.9 -> 11.9 mm, vias 0 -> 2
- net /USB_D+: track 12.5 -> 13.6 mm, vias 2 -> 0
- net Net-(R7-Pad2): track 11.7 -> 12.2 mm
- net /RUN: track 17.9 -> 18.5 mm
