File: eurorack/accessories/chordata/_autosave-chordata 2.kicad_pcb (KiCad board)
At the start: 2 copper layers, 20.3 x 45.7 mm, 43 parts, among them J1 USB_C_Receptacle_USB2.0, J2 Conn_02x05_Odd_Even, J3 Conn_01x18, J4 Conn_01x18, SW1 SW_Push, SW2 SW_Push, U1 AMS1117-3.3, U2 RP2040, U3 W25Q128JVS, Y1 Crystal_GND24

Commit message: chordata v2 final layout
Parts:
- G1: value LOGO -> Artwork; footprint LOGO -> Pale Slim Ghost:logo 12mm
- moved JP1 0.76 mm to (106.9, 61.7)
- moved G1 0.74 mm to (101.2, 62.5)
- moved D3 0.28 mm to (98.7, 65.8)
- moved R10 0.28 mm to (101.4, 65.8)
Other:
- board text added: "Boot"
- board text added: "Chordata v2 · Sept 2022"
- board text added: "Reset"
- board text removed: "Chordata v2 · Oct 2022"
- board text removed: "boot"
- board text removed: "reset"
