File: eurorack/panels/chord-organ/chord-organ.kicad_pcb (KiCad board)
At the start: 4 copper layers, 20.3 x 128.5 mm, 17 parts

Commit message: final chord organ design
Parts:
- added @HOLE5: , , F.Cu at (165.5, 113.8)
Other:
- board text added: "JLCJLCJLCJLC"
Changed lines of the file:
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@@
+  )
+  (footprint "" (layer "F.Cu")
+    (at 165.481 113.792 90)
+    (fp_text reference "@HOLE5" (at 0 0 90) (layer "F.SilkS") hide
+      (effects (font (size 1.27 1.27) (thickness 0.15)))
+    )
+    (fp_text value "" (at 0 0 90) (layer "F.SilkS")
+      (effects (font (size 1.27 1.27) (thickness 0.15)))
+    )
   )
   (footprint "" (layer "F.Cu")
@@
   (gr_circle (center 152.4 137.414) (end 156.972 137.414) (layer "User.1") (width 0.1) (fill none))
   (gr_circle (center 147.32 91.186) (end 153.416 91.186) (layer "User.1") (width 0.1) (fill none))
+  (gr_text "JLCJLCJLCJLC" (at 147.447 162.433) (layer "B.SilkS")
+    (effects (font (size 1 1) (thickness 0.15)) (justify mirror))
+  )
   (gr_text "Chord" (at 142.24 143.51) (layer "F.SilkS")
     (effects (font (size 2 1.6) (thickness 0.15)))
