File: eurorack/accessories/ants-psu/ants-psu.kicad_sch (KiCad schematic)
At the start: 9 parts, among them J1 PJ-064B, J2 Conn_02x08_Odd_Even, SW1 SW_SPST

Commit message: ants v2 final design
Parts:
- removed J1: PJ-064B, Pale Slim Ghost:CUI_PJ-064B, symbol PJ-064B:PJ-064B
- removed J2: Conn_02x08_Odd_Even, Pale Slim Ghost:PinHeader_Shrouded_2x08_P2.54mm_Vertical, symbol Connector_Generic:Conn_02x08_Odd_Even
- removed SW1: SW_SPST, Pale Slim Ghost:Mini Toggle Switch SPDT, symbol Switch:SW_SPST
- added C2, C3: 47μ, Capacitor_SMD:CP_Elec_5x4.5, symbol Device:C_Polarized
- added H1, H2, H3, H4: MountingHole, MountingHole:MountingHole_3.2mm_M3, symbol Mechanical:MountingHole
- added J1, J2: Conn_01x04, Pale Slim Ghost:Molex_KK-254_AE-6410-04A_1x04_P2.54mm_Horizontal, symbol Connector_Generic:Conn_01x04
- added J17: Conn_01x06, Pale Slim Ghost:Molex_KK-254_AE-6410-06A_1x06_P2.54mm_Horizontal, symbol Connector_Generic:Conn_01x06
- D1: value LED -> red
- D2: value LED -> blue
Connections:
- net +12V: now also R1.2, C2.1, J17.2 (Pin_2), J17.5 (Pin_5); no longer R1.1
- net -12V: now also C3.2, J17.1 (Pin_1), J17.6 (Pin_6)
- net Earth: now also J1.2 (Pin_2), J1.3 (Pin_3), J2.2 (Pin_2), J2.3 (Pin_3)
- net GND: now also R2.2, C2.2, C3.1, J17.3 (Pin_3), J17.4 (Pin_4); no longer R2.1
- net at D1.2 (A): now also R1.1; no longer R1.2
- net at D2.2 (A): now also R2.1; no longer R2.2
- net VIN renamed VDC
- net VDC: now also J1.1 (Pin_1), J1.4 (Pin_4), J2.1 (Pin_1), J2.4 (Pin_4)
- no-connect marks 0 -> 1
Other:
- moved on the sheet: C1
