File: eurorack/accessories/bus/bus.kicad_pcb (KiCad board)
At the start: 2 copper layers, 241.9 x 26.7 mm, 22 parts, among them J1 Conn_02x08_Odd_Even, J10 Conn_02x08_Odd_Even, J11 Conn_02x08_Odd_Even, J12 Conn_02x08_Odd_Even, J13 Conn_02x08_Odd_Even, J14 Conn_02x08_Odd_Even, J15 Conn_02x08_Odd_Even, J16 Conn_02x08_Odd_Even, J2 Conn_02x08_Odd_Even, J3 Conn_02x08_Odd_Even, J4 Conn_02x08_Odd_Even, J5 Conn_02x08_Odd_Even, J6 Conn_02x08_Odd_Even, J7 Conn_02x08_Odd_Even, J8 Conn_02x08_Odd_Even, J9 Conn_02x08_Odd_Even

Commit message: bus v2
Parts:
- removed G*** (x2): LOGO, LOGO
- removed REF** (x4): MountingHole_3.2mm_M3, MountingHole:MountingHole_3.2mm_M3
- added H1: MountingHole, MountingHole:MountingHole_3.2mm_M3, F.Cu at (25.4, 73.1)
- added H2: MountingHole, MountingHole:MountingHole_3.2mm_M3, F.Cu at (25.4, 93.3)
- added H3: MountingHole, MountingHole:MountingHole_3.2mm_M3, F.Cu at (261.0, 73.0)
- added H4: MountingHole, MountingHole:MountingHole_3.2mm_M3, F.Cu at (261.0, 93.3)
- added J17: Conn_01x06, Pale Slim Ghost:Molex_KK-254_AE-6410-06A_1x06_P2.54mm_Horizontal, F.Cu at (32.4, 87.0)
- added J18: Conn_01x06, Pale Slim Ghost:Molex_KK-254_AE-6410-06A_1x06_P2.54mm_Horizontal, F.Cu at (254.0, 79.2)
Routing:
- net +12V: track 389.4 -> 430.8 mm
- net -12V: track 404.9 -> 427.4 mm
- net Gate: track 406.5 -> 404.4 mm
Other:
- board text added: "bus board v2"
- board text added: "march 2023"
