File: eurorack/accessories/bus/bus.kicad_sch (KiCad schematic)
At the start: 16 parts, among them J1 Conn_02x08_Odd_Even, J10 Conn_02x08_Odd_Even, J11 Conn_02x08_Odd_Even, J12 Conn_02x08_Odd_Even, J13 Conn_02x08_Odd_Even, J14 Conn_02x08_Odd_Even, J15 Conn_02x08_Odd_Even, J16 Conn_02x08_Odd_Even, J2 Conn_02x08_Odd_Even, J3 Conn_02x08_Odd_Even, J4 Conn_02x08_Odd_Even, J5 Conn_02x08_Odd_Even, J6 Conn_02x08_Odd_Even, J7 Conn_02x08_Odd_Even, J8 Conn_02x08_Odd_Even, J9 Conn_02x08_Odd_Even

Commit message: bus v2
Parts:
- added H1, H2, H3, H4: MountingHole, MountingHole:MountingHole_3.2mm_M3, symbol Mechanical:MountingHole
- added J17, J18: Conn_01x06, Pale Slim Ghost:Molex_KK-254_AE-6410-06A_1x06_P2.54mm_Horizontal, symbol Connector_Generic:Conn_01x06
Connections:
- net +12V: now also J17.2 (Pin_2), J17.5 (Pin_5), J18.2 (Pin_2), J18.5 (Pin_5)
- net -12V: now also J17.1 (Pin_1), J17.6 (Pin_6), J18.1 (Pin_1), J18.6 (Pin_6)
- net GND: now also J17.3 (Pin_3), J17.4 (Pin_4), J18.3 (Pin_3), J18.4 (Pin_4)
