File: eurorack/modules/spiders/spiders.kicad_pcb (KiCad board)
At the start: 2 copper layers, 66 x 128.3 mm, 116 parts, among them J1 AudioJack2_SwitchT, J10 Conn_01x08_Female, J11 Conn_02x08_Odd_Even, J12 Conn_02x08_Odd_Even, J2 AudioJack2_SwitchT, J3 AudioJack2_SwitchT, J4 AudioJack2_SwitchT, J5 AudioJack2_SwitchT, J6 AudioJack2_SwitchT, J7 AudioJack2_SwitchT, J8 AudioJack2_SwitchT, J9 Conn_01x08_Male, SW1 SW_Push_LED, SW2 SW_Push_LED, SW3 SW_Push_LED, SW4 SW_Push_LED, SW5 SW_Push_LED, SW6 SW_Push_LED, SW7 SW_Push_LED, SW8 SW_Push_LED, U1 TL074, U10 Chordata, U2 TMUX8212, U3 TL074, U4 TMUX8212, U5 TL074, U6 TMUX8212, U8 TMUX8212

Commit message: spiders tweaks
Parts:
- D1, D2, D3, D4, D5, D6, D7, D8: footprint Diode_SMD:D_0805_2012Metric -> Diode_SMD:D_SOD-323_HandSoldering
Other:
- board text added: "april 2023"
- board text added: "spiders v1.1"
- board text removed: "Pale Slim Ghost Synthesisers"
- board text removed: "Spiders v1 January 2023"

Commit message: spiders v1 files
Parts:
- removed B1, B2: Mousebite, Pale Slim Ghost:mousebite-2.54x5.08mm
- removed G*** (x2): LOGO, LOGO
- removed H10, H11, H12, H13, H14, H15, H16, H17, H18, H3, H4, H5, H6, H7, H8, H9: MountingHole, Pale Slim Ghost:hole 6mm (jack panel)
- removed H19, H20: MountingHole, Pale Slim Ghost:eurorack panel mounting slot
- removed H2: MountingHole, MountingHole:MountingHole_2.2mm_M2
Connections:
- U10 pad 17: +12V -> GND
- U10 pad 18: GND -> +12V
- U10 pad 19: GND -> -12V
- U10 pad 20: -12V -> GND
Routing:
- net -12V: track 85.4 -> 88.0 mm
- net +12V: track 85.3 -> 87.8 mm
- removed copper zone on B.Cu, net (none)
- removed copper zone on F.Cu, net (none)
Other:
- board size 66 x 128.3 mm -> 43.2 x 110.4 mm
