File: eurorack/modules/spiders/spiders.kicad_sch (KiCad schematic)
At the start: 115 parts, among them J1 AudioJack2_SwitchT, J10 Conn_01x08_Female, J11 Conn_02x08_Odd_Even, J12 Conn_02x08_Odd_Even, J2 AudioJack2_SwitchT, J3 AudioJack2_SwitchT, J4 AudioJack2_SwitchT, J5 AudioJack2_SwitchT, J6 AudioJack2_SwitchT, J7 AudioJack2_SwitchT, J8 AudioJack2_SwitchT, J9 Conn_01x08_Male, SW1 SW_Push_LED, SW2 SW_Push_LED, SW3 SW_Push_LED, SW4 SW_Push_LED, SW5 SW_Push_LED, SW6 SW_Push_LED, SW7 SW_Push_LED, SW8 SW_Push_LED, U1 TL074, U10 Chordata, U2 TMUX8212, U3 TL074, U4 TMUX8212, U5 TL074, U6 TMUX8212, U8 TMUX8212

Commit message: spiders tweaks
Parts:
- D1, D2, D3, D4, D5, D6, D7, D8: footprint Diode_SMD:D_0805_2012Metric -> Diode_SMD:D_SOD-323_HandSoldering

Commit message: spiders v1 files
Parts:
- removed B1, B2: Mousebite, Pale Slim Ghost:mousebite-2.54x5.08mm, symbol Pale Slim Ghost:Mousebite
- removed H10, H11, H12, H13, H14, H15, H16, H17, H18, H3, H4, H5, H6, H7, H8, H9: MountingHole, Pale Slim Ghost:hole 6mm (jack panel), symbol Mechanical:MountingHole
- removed H19, H20: MountingHole, Pale Slim Ghost:eurorack panel mounting slot, symbol Mechanical:MountingHole
- removed H2: MountingHole, MountingHole:MountingHole_2.2mm_M2, symbol Mechanical:MountingHole
Connections:
- net +12V: now also U10.18 (+12V); no longer U10.17 (+12V)
- net -12V: now also U10.19 (-12V); no longer U10.20 (-12V)
- net GND: now also U10.17 (GND), U10.20 (GND); no longer U10.18 (GND), U10.19 (GND)
