File: eurorack/modules/bats/bats.kicad_pcb (KiCad board)
At the start: 2 copper layers, 30.5 x 65 mm, 29 parts, among them J1 Conn_02x05_Odd_Even, J2 AudioJack2_SwitchT, J3 AudioJack2_SwitchT, U1 TL072, U2 TMUX6219, U3 74LVC1G74, U4 MIC5219-3.3YM5

Commit message: bats v2
Parts:
- removed G***: LOGO, LOGO
- added D2: red, LED_SMD:LED_0805_2012Metric_Pad1.15x1.40mm_HandSolder, F.Cu at (142.0, 72.0)
- added G1, G2: LOGO, LOGO, F.Cu at (134.2, 38.1)
- added H6: MountingHole, Pale Slim Ghost:hole 3mm (below jack), F.Cu at (143.0, 38.0)
- added L1: LED_Lightpipe, Pale Slim Ghost:VBL Lightpipe, F.Cu at (143.0, 72.0)
- C1, C2, C4, C5, C6: value C -> 100n
- C3, C7: value C_Polarized -> 10u; moved to F.Cu
- D1: value LED_Dual_Bidirectional -> blue; footprint LED_THT:LED_D3.0mm_Clear -> LED_SMD:LED_0805_2012Metric_Pad1.15x1.40mm_HandSolder
- R1, R2: value R -> 20k
- R3: value R -> 1k
- R4: value R -> 10k
- R5: value R -> 560
- RV1: footprint Pale Slim Ghost:P170NP1 Switch Potentiometer -> Pale Slim Ghost:PRS11R Momentary Switch Potentiometer
- moved C3 24.7 mm to (146.8, 71.9), turned to -90 degrees
- moved U4 20.4 mm to (129.0, 62.5), turned to 180 degrees
- moved C8 19.7 mm to (124.2, 62.5), turned to 180 degrees
- moved R2 18.4 mm to (122.3, 75.6), turned to 90 degrees
- moved C5 18.3 mm to (123.8, 78.9), turned to 90 degrees
- moved J1 18.2 mm to (141.7, 71.9), turned to -90 degrees
- moved C7 17.5 mm to (137.9, 71.9), turned to -90 degrees
- moved C4 16.2 mm to (123.7, 67.2), turned to 180 degrees
- moved R1 14.0 mm to (123.8, 75.6), turned to -90 degrees
- moved U3 12.7 mm to (128.3, 67.7), turned to 180 degrees
- moved C6 11.8 mm to (123.7, 69.6), turned to 0 degrees
- moved C1 10.1 mm to (132.7, 78.9), turned to -90 degrees
- moved R4 8.93 mm to (133.2, 63.4)
- moved U1 7.49 mm to (128.3, 72.3), turned to 0 degrees
- moved R3 7.25 mm to (136.5, 81.5)
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Connections:
- R5 pad 1: Net-(R5-Pad1) -> Net-(D1-Pad1)
- U1 pad 5: Net-(R5-Pad1) -> GND
- U1 pad 6: Net-(D1-Pad2) -> Net-(D1-Pad1)
- U1 pad 7: Net-(D1-Pad1) -> Net-(D1-Pad2)
Routing:
- net +12V: track 7.69 -> 53.4 mm, vias 2 -> 1
- net GND: track 15.3 -> 0.00 mm, vias 9 -> 0
- net Net-(RV1-PadS2): track 15.7 -> 2.03 mm, vias 1 -> 0
- net Net-(J2-PadT): track 41.1 -> 48.0 mm, vias 1 -> 0
- net +3.3V: track 15.5 -> 10.8 mm
- net -12V: track 37.1 -> 32.5 mm, vias 4 -> 3
- net switch: track 7.08 -> 11.2 mm, vias 0 -> 2
- net Net-(J3-PadT): track 7.66 -> 11.6 mm
- net Net-(D1-Pad1): track 13.2 -> 16.7 mm, vias 0 -> 1
- net Net-(R1-Pad1): track 7.76 -> 5.47 mm
- net Net-(J2-PadTN): track 4.13 -> 6.21 mm
- net Net-(R5-Pad1): track 1.85 -> 0.00 mm
- net Net-(U1-Pad3): track 8.29 -> 6.63 mm, vias 2 -> 0
- net Net-(D1-Pad2): track 15.1 -> 16.3 mm, vias 0 -> 1
- net Net-(RV1-Pad2): track 5.78 -> 4.57 mm
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- removed copper zone on B.Cu, net +12V
Other:
- board text added: "Bats v2 • Nov 2022"
- board text added: "JLCJLCJLCJLC"

Commit message: assorted changes ig from opening things in kicad 7
Parts:
- removed H6: MountingHole, Pale Slim Ghost:hole 3mm (below jack)
- removed L1: LED_Lightpipe, Pale Slim Ghost:VBL Lightpipe
- C1, C2, C4, C5, C6: footprint Capacitor_SMD:C_0603_1608Metric_Pad1.08x0.95mm_HandSolder -> Capacitor_SMD:C_0805_2012Metric_Pad1.18x1.45mm_HandSolder
- R1, R2, R3, R4, R5: footprint Resistor_SMD:R_0603_1608Metric_Pad0.98x0.95mm_HandSolder -> Resistor_SMD:R_0805_2012Metric_Pad1.20x1.40mm_HandSolder
- moved C1 0.65 mm to (132.8, 79.5)
- moved C5 0.65 mm to (123.7, 79.5)
- moved R2 0.64 mm to (121.7, 75.6)
- moved C6 0.46 mm to (123.4, 69.2)
- moved C4 0.36 mm to (123.4, 66.9)
- moved C2 0.13 mm to (132.8, 75.6)
- moved R1 0.13 mm to (123.7, 75.6)
Routing:
- net Net-(R1-Pad2): track 41.0 -> 42.7 mm
- net Net-(J2-PadT): track 48.0 -> 49.6 mm
- net +12V: track 53.4 -> 54.6 mm
