File: eurorack/modules/bats/bats.kicad_sch (KiCad schematic)
At the start: 28 parts, among them J1 Conn_02x05_Odd_Even, J2 AudioJack2_SwitchT, J3 AudioJack2_SwitchT, U1 TL072, U2 TMUX6219, U3 74LVC1G74, U4 MIC5219-3.3YM5

Commit message: bats v2
Parts:
- removed D1: LED_Dual_Bidirectional, LED_THT:LED_D3.0mm_Clear, symbol Device:LED_Dual_Bidirectional
- added D1: blue, LED_SMD:LED_0805_2012Metric_Pad1.15x1.40mm_HandSolder, symbol Device:LED
- added D2: red, LED_SMD:LED_0805_2012Metric_Pad1.15x1.40mm_HandSolder, symbol Device:LED
- added G1, G2: Artwork, symbol Pale Slim Ghost:Artwork
- added H6: MountingHole, Pale Slim Ghost:hole 3mm (below jack), symbol Mechanical:MountingHole
- added L1: LED_Lightpipe, Pale Slim Ghost:VBL Lightpipe, symbol Pale Slim Ghost:LED_Lightpipe
- C1, C2, C4, C5, C6: value C -> 100n
- C3, C7: value C_Polarized -> 10u
- R1, R2: value R -> 20k
- R3: value R -> 1k
- R4: value R -> 10k
- R5: value R -> 560
- RV1: footprint Pale Slim Ghost:P170NP1 Switch Potentiometer -> Pale Slim Ghost:PRS11R Momentary Switch Potentiometer; Part # (none) -> P170SP1-QC15BR10K
Connections:
- net GND: now also U1.5 (+)
- net at R5.1: now also U1.6 (-), D1.1 (K), D2.2 (A); no longer U1.5 (+)
- net at U1.7: now also D1.2 (A), D2.1 (K)
Other:
- moved on the sheet: U1B

Commit message: assorted changes ig from opening things in kicad 7
Parts:
- removed H6: MountingHole, Pale Slim Ghost:hole 3mm (below jack), symbol Mechanical:MountingHole
- removed L1: LED_Lightpipe, Pale Slim Ghost:VBL Lightpipe, symbol Pale Slim Ghost:LED_Lightpipe
- C1, C2, C4, C5, C6: footprint Capacitor_SMD:C_0603_1608Metric_Pad1.08x0.95mm_HandSolder -> Capacitor_SMD:C_0805_2012Metric_Pad1.18x1.45mm_HandSolder
- R1, R2, R3, R4, R5: footprint Resistor_SMD:R_0603_1608Metric_Pad0.98x0.95mm_HandSolder -> Resistor_SMD:R_0805_2012Metric_Pad1.20x1.40mm_HandSolder
Changed lines of the file:
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@@
     (property "Reference" "R1" (id 0) (at 147.701 68.58 90))
     (property "Value" "20k" (id 1) (at 147.701 71.12 90))
-    (property "Footprint" "Resistor_SMD:R_0603_1608Metric_Pad0.98x0.95mm_HandSolder" (id 2) (at 147.701 76.073 90)
+    (property "Footprint" "Resistor_SMD:R_0805_2012Metric_Pad1.20x1.40mm_HandSolder" (id 2) (at 147.701 76.073 90)
       (effects (font (size 1.27 1.27)) hide)
     )
@@
     (pin "1")
     (pin "2")
-  )
-  (symbol (lib_id "Mechanical:MountingHole") (at 154.051 125.095 0) (unit 1)
-    (in_bom yes) (on_board yes) (fields_autoplaced)
-    (property "Reference" "H6" (id 0) (at 157.48 123.8249 0)
-      (effects (font (size 1.27 1.27)) (justify left))
-    )
-    (property "Value" "MountingHole" (id 1) (at 157.48 126.3649 0)
-      (effects (font (size 1.27 1.27)) (justify left))
-    )
-    (property "Footprint" "Pale Slim Ghost:hole 3mm (below jack)" (id 2) (at 154.051 125.095 0)
-      (effects (font (size 1.27 1.27)) hide)
-    )
-    (property "Datasheet" "~" (id 3) (at 154.051 125.095 0)
-      (effects (font (size 1.27 1.27)) hide)
-    )
   )
   (symbol (lib_id "Mechanical:MountingHole") (at 95.504 28.829 0) (unit 1)
@@
       (effects (font (size 1.27 1.27)) (justify left))
     )
-    (property "Footprint" "Capacitor_SMD:C_0603_1608Metric_Pad1.08x0.95mm_HandSolder" (id 2) (at 185.6232 37.973 0)
+    (property "Footprint" "Capacitor_SMD:C_0805_2012Metric_Pad1.18x1.45mm_HandSolder" (id 2) (at 185.6232 37.973 0)
       (effects (font (size 1.27 1.27)) hide)
     )
@@
       (effects (font (size 1.27 1.27)) (justify left))
     )
-    (property "Footprint" "Capacitor_SMD:C_0603_1608Metric_Pad1.08x0.95mm_HandSolder" (id 2) (at 185.6232 45.593 0)
+    (property "Footprint" "Capacitor_SMD:C_0805_2012Metric_Pad1.18x1.45mm_HandSolder" (id 2) (at 185.6232 45.593 0)
       (effects (font (size 1.27 1.27)) hide)
     )
@@
       (effects (font (size 1.27 1.27)) (justify right))
     )
-    (property "Footprint" "Resistor_SMD:R_0603_1608Metric_Pad0.98x0.95mm_HandSolder" (id 2) (at 112.268 89.027 90)
+    (property "Footprint" "Resistor_SMD:R_0805_2012Metric_Pad1.20x1.40mm_HandSolder" (id 2) (at 112.268 89.027 90)
       (effects (font (size 1.27 1.27)) hide)
     )
@@
     (pin "8")
   )
-  (symbol (lib_id "Pale Slim Ghost:LED_Lightpipe") (at 159.258 128.143 0) (unit 1)
-    (in_bom yes) (on_board yes) (fields_autoplaced)
-    (property "Reference" "L1" (id 0) (at 161.29 122.4229 0)
-      (effects (font (size 1.27 1.27)) (justify left))
-    )
-    (property "Value" "LED_Lightpipe" (id 1) (at 161.29 124.9629 0)
-      (effects (font (size 1.27 1.27)) (justify left))
-    )
-    (property "Footprint" "Pale Slim Ghost:VBL Lightpipe" (id 2) (at 159.258 128.143 0)
-      (effects (font (size 1.27 1.27)) hide)
-    )
-    (property "Datasheet" "" (id 3) (at 159.258 128.143 0)
-      (effects (font (size 1.27 1.27)) hide)
-    )
-  )
   (symbol (lib_id "Device:LED") (at 167.767 111.379 0) (unit 1)
     (in_bom yes) (on_board yes) (fields_autoplaced)
@@
       (effects (font (size 1.27 1.27)) (justify left))
     )
-    (property "Footprint" "Resistor_SMD:R_0603_1608Metric_Pad0.98x0.95mm_HandSolder" (id 2) (at 157.226 93.726 90)
+    (property "Footprint" "Resistor_SMD:R_0805_2012Metric_Pad1.20x1.40mm_HandSolder" (id 2) (at 157.226 93.726 90)
       (effects (font (size 1.27 1.27)) hide)
     )
@@
     (property "Reference" "R3" (id 0) (at 159.258 78.74 90))
     (property "Value" "1k" (id 1) (at 159.258 81.28 90))
-    (property "Footprint" "Resistor_SMD:R_0603_1608Metric_Pad0.98x0.95mm_HandSolder" (id 2) (at 159.258 86.995 90)
+    (property "Footprint" "Resistor_SMD:R_0805_2012Metric_Pad1.20x1.40mm_HandSolder" (id 2) (at 159.258 86.995 90)
       (effects (font (size 1.27 1.27)) hide)
     )
@@
       (effects (font (size 1.27 1.27)) (justify left))
     )
-    (property "Footprint" "Capacitor_SMD:C_0603_1608Metric_Pad1.08x0.95mm_HandSolder" (id 2) (at 253.4412 38.1 0)
+    (property "Footprint" "Capacitor_SMD:C_0805_2012Metric_Pad1.18x1.45mm_HandSolder" (id 2) (at 253.4412 38.1 0)
       (effects (font (size 1.27 1.27)) hide)
     )
@@
     (property "Reference" "R2" (id 0) (at 136.398 76.2 90))
     (property "Value" "20k" (id 1) (at 136.398 78.74 90))
-    (property "Footprint" "Resistor_SMD:R_0603_1608Metric_Pad0.98x0.95mm_HandSolder" (id 2) (at 136.398 84.455 90)
+    (property "Footprint" "Resistor_SMD:R_0805_2012Metric_Pad1.20x1.40mm_HandSolder" (id 2) (at 136.398 84.455 90)
       (effects (font (size 1.27 1.27)) hide)
     )
@@
       (effects (font (size 1.27 1.27)) (justify left))
     )
-    (property "Footprint" "Capacitor_SMD:C_0603_1608Metric_Pad1.08x0.95mm_HandSolder" (id 2) (at 253.4412 45.72 0)
+    (property "Footprint" "Capacitor_SMD:C_0805_2012Metric_Pad1.18x1.45mm_HandSolder" (id 2) (at 253.4412 45.72 0)
       (effects (font (size 1.27 1.27)) hide)
     )
@@
       (effects (font (size 1.27 1.27)) (justify left))
     )
-    (property "Footprint" "Capacitor_SMD:C_0603_1608Metric_Pad1.08x0.95mm_HandSolder" (id 2) (at 227.6602 42.926 0)
+    (property "Footprint" "Capacitor_SMD:C_0805_2012Metric_Pad1.18x1.45mm_HandSolder" (id 2) (at 227.6602 42.926 0)
       (effects (font (size 1.27 1.27)) hide)
     )
@@
     )
     (path "/20d9c372-bc05-4a2f-8b1b-d56f2a2c6d3c"
-      (reference "C1") (unit 1) (value "100n") (footprint "Capacitor_SMD:C_0603_1608Metric_Pad1.08x0.95mm_HandSolder")
+      (reference "C1") (unit 1) (value "100n") (footprint "Capacitor_SMD:C_0805_2012Metric_Pad1.18x1.45mm_HandSolder")
     )
     (path "/a5d17d36-b77d-4e1f-8eb4-4ab2166afb9a"
-      (reference "C2") (unit 1) (value "100n") (footprint "Capacitor_SMD:C_0603_1608Metric_Pad1.08x0.95mm_HandSolder")
+      (reference "C2") (unit 1) (value "100n") (footprint "Capacitor_SMD:C_0805_2012Metric_Pad1.18x1.45mm_HandSolder")
     )
     (path "/b61ecb1e-cdc3-4037-9286-8cd5ae6f8cd8"
@@
     )
     (path "/dee1d876-7112-4196-ba01-2a89706d4746"
-      (reference "C4") (unit 1) (value "100n") (footprint "Capacitor_SMD:C_0603_1608Metric_Pad1.08x0.95mm_HandSolder")
+      (reference "C4") (unit 1) (value "100n") (footprint "Capacitor_SMD:C_0805_2012Metric_Pad1.18x1.45mm_HandSolder")
     )
     (path "/3699e5f4-721a-4c84-95cb-fa2a93d669b0"
-      (reference "C5") (unit 1) (value "100n") (footprint "Capacitor_SMD:C_0603_1608Metric_Pad1.08x0.95mm_HandSolder")
+      (reference "C5") (unit 1) (value "100n") (footprint "Capacitor_SMD:C_0805_2012Metric_Pad1.18x1.45mm_HandSolder")
     )
     (path "/ca18cbcb-420f-4027-af6a-3ceac717f696"
-      (reference "C6") (unit 1) (value "100n") (footprint "Capacitor_SMD:C_0603_1608Metric_Pad1.08x0.95mm_HandSolder")
+      (reference "C6") (unit 1) (value "100n") (footprint "Capacitor_SMD:C_0805_2012Metric_Pad1.18x1.45mm_HandSolder")
     )
     (path "/9a462d07-09df-43cc-8043-31e9c6a5a423"
@@
       (reference "H5") (unit 1) (value "MountingHole") (footprint "Pale Slim Ghost:hole 6.5mm (potentiometer panel)")
     )
-    (path "/1456dbe9-af4b-4d03-ab17-5c3e37bf40f9"
-      (reference "H6") (unit 1) (value "MountingHole") (footprint "Pale Slim Ghost:hole 3mm (below jack)")
-    )
     (path "/0f7a4462-b90c-479b-b7a9-0c7aea7b4f55"
       (reference "J1") (unit 1) (value "Conn_02x05_Odd_Even") (footprint "Connector_PinHeader_2.54mm:PinHeader_2x05_P2.54mm_Vertical_SMD")
@@
       (reference "J3") (unit 1) (value "AudioJack2_SwitchT") (footprint "Pale Slim Ghost:Jack_3.5mm_QingPu_WQP-PJ398SM_Vertical")
     )
-    (path "/544a08ab-acb7-4412-823f-333ed66d3b11"
-      (reference "L1") (unit 1) (value "LED_Lightpipe") (footprint "Pale Slim Ghost:VBL Lightpipe")
-    )
     (path "/136170b2-a3d7-4989-9b70-fa58dfe81658"
-      (reference "R1") (unit 1) (value "20k") (footprint "Resistor_SMD:R_0603_1608Metric_Pad0.98x0.95mm_HandSolder")
+      (reference "R1") (unit 1) (value "20k") (footprint "Resistor_SMD:R_0805_2012Metric_Pad1.20x1.40mm_HandSolder")
     )
     (path "/c1a39f3d-9ac8-4654-8803-a19e27a102fb"
-      (reference "R2") (unit 1) (value "20k") (footprint "Resistor_SMD:R_0603_1608Metric_Pad0.98x0.95mm_HandSolder")
+      (reference "R2") (unit 1) (value "20k") (footprint "Resistor_SMD:R_0805_2012Metric_Pad1.20x1.40mm_HandSolder")
     )
     (path "/892925bf-1354-45ff-bd11-b17e07e60b53"
-      (reference "R3") (unit 1) (value "1k") (footprint "Resistor_SMD:R_0603_1608Metric_Pad0.98x0.95mm_HandSolder")
+      (reference "R3") (unit 1) (value "1k") (footprint "Resistor_SMD:R_0805_2012Metric_Pad1.20x1.40mm_HandSolder")
     )
     (path "/3db25457-c686-45de-9fa9-dddef8f443d1"
-      (reference "R4") (unit 1) (value "10k") (footprint "Resistor_SMD:R_0603_1608Metric_Pad0.98x0.95mm_HandSolder")
+      (reference "R4") (unit 1) (value "10k") (footprint "Resistor_SMD:R_0805_2012Metric_Pad1.20x1.40mm_HandSolder")
     )
     (path "/73782606-bcef-485b-b3cd-7a22ce77e842"
-      (reference "R5") (unit 1) (value "560") (footprint "Resistor_SMD:R_0603_1608Metric_Pad0.98x0.95mm_HandSolder")
+      (reference "R5") (unit 1) (value "560") (footprint "Resistor_SMD:R_0805_2012Metric_Pad1.20x1.40mm_HandSolder")
     )
     (path "/09d48e28-1ef8-4a2d-b093-27d38820531c"
