File: standalone/encoders/encoders front panel.kicad_pcb (KiCad board)
At the start: 2 copper layers, 78.5 x 35.6 mm, 6 parts

Commit message: add ocelots
Parts:
- removed G***: LOGO, LOGO
- removed H1, H2, H3, H4: MountingHole, MountingHole:MountingHole_2.2mm_M2
- removed REF**: hole 9mm (encoder panel), Pale Slim Ghost:hole 9mm (encoder panel)
Other:
- board size 78.5 x 35.6 mm -> 55.9 x 55.9 mm
