File: standalone/encoders/encoders.kicad_sch (KiCad schematic)
At the start: 20 parts, among them SW1 RotaryEncoder_Switch, SW2 RotaryEncoder_Switch, SW3 RotaryEncoder_Switch, SW4 RotaryEncoder_Switch, SW5 SW_SPDT, SW6 SW_Push, U1 ProMicro

Commit message: add ocelots
Parts:
- removed BT1: Battery_Cell, Connector_JST:JST_PH_S2B-PH-K_1x02_P2.00mm_Horizontal, symbol Device:Battery_Cell
- removed SW5: SW_SPDT, Pale Slim Ghost:EG1247, symbol Switch:SW_SPDT
- removed SW6: SW_Push, Pale Slim Ghost:MJPT1117 Tactile Switch, symbol Switch:SW_Push
- added D2: SK6812, LED_SMD:LED_SK6812_PLCC4_5.0x5.0mm_P3.2mm, symbol LED:SK6812
- C1, C2, C3, C4, C5, C6, C7, C8: footprint Capacitor_THT:C_Disc_D5.0mm_W2.5mm_P5.00mm -> Capacitor_SMD:C_0805_2012Metric_Pad1.18x1.45mm_HandSolder
- H1, H2, H3, H4: footprint MountingHole:MountingHole_2.2mm_M2 -> MountingHole:MountingHole_2.2mm_M2_Pad_TopOnly; now left out of the parts list
- SW1, SW2, SW3, SW4, U1: now left out of the parts list
Connections:
- net Encoder 1 A: now also U1.18 (F6/A1); no longer U1.6 (3/D0/SCL)
- net Encoder 1 B: now also U1.17 (F7/A0); no longer U1.19 (F5/A2)
- net Encoder 1 Switch: now also SW1.S1, U1.19 (F5/A2); no longer SW1.S2, U1.20 (F4/A3)
- net Encoder 2 B: now also U1.7 (4/D4); no longer U1.17 (F7/A0)
- net Encoder 2 Switch: now also U1.6 (3/D0/SCL); no longer U1.18 (F6/A1)
- net Encoder 3 A: now also U1.14 (B2/16); no longer U1.10 (7/E6)
- net Encoder 3 Switch: now also U1.13 (B6/10); no longer U1.16 (B1/15)
- net Encoder 4 A: now also U1.10 (7/E6); no longer U1.12 (9/B5)
- net Encoder 4 B: now also U1.11 (8/B4); no longer U1.13 (B6/10)
- net Encoder 4 Switch: now also SW4.S1, U1.12 (9/B5); no longer SW4.S2, U1.14 (B2/16)
- net GND: now also SW1.S2, SW4.S2, D2.1 (VSS); no longer SW1.S1, SW4.S1
- net LED: now reaches U1.5 (2/D1/SDA)
- net LED: now also D2.2 (DIN)
- net +5V renamed +3.3V
- net +3.3V: now also D2.3 (VDD)
