File: eurorack/accessories/screen/screen.kicad_sch (KiCad schematic)
At the start: 11 parts, among them J1 Conn_01x04

Commit message: jan 24
Parts:
- J1, U1: now left out of the parts list
- R1: value 310r -> 310K
Connections:
- net +3.3V: now also U1.9 (~{RES})
Changed lines of the file:
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@@
+    )
+  )
+  (symbol (lib_id "power:+3.3V") (at 103.251 75.057 90) (unit 1)
+    (in_bom yes) (on_board yes) (dnp no) (fields_autoplaced)
+    (property "Reference" "#PWR015" (at 107.061 75.057 0)
+      (effects (font (size 1.27 1.27)) hide)
+    )
+    (property "Value" "+3.3V" (at 99.06 75.692 90)
+      (effects (font (size 1.27 1.27)) (justify left))
+    )
+    (property "Footprint" "" (at 103.251 75.057 0)
+      (effects (font (size 1.27 1.27)) hide)
+    )
+    (property "Datasheet" "" (at 103.251 75.057 0)
+      (effects (font (size 1.27 1.27)) hide)
+    )
+    (pin "1")
+    (instances
+      (project "screen"
+        (path "/c918c880-43c2-4652-b720-5af29f34729b"
+          (reference "#PWR015") (unit 1)
+        )
+      )
     )
   )
@@
       (effects (font (size 1.27 1.27)))
     )
-    (property "Value" "310r" (at 99.441 80.01 90)
+    (property "Value" "310K" (at 99.441 80.01 90)
       (effects (font (size 1.27 1.27)))
     )
@@
   )
   (symbol (lib_id "Connector_Generic:Conn_01x04") (at 79.883 33.782 0) (unit 1)
-    (in_bom yes) (on_board yes) (dnp no) (fields_autoplaced)
+    (in_bom no) (on_board yes) (dnp no) (fields_autoplaced)
     (property "Reference" "J1" (at 82.55 34.417 0)
       (effects (font (size 1.27 1.27)) (justify left))
@@
   )
   (symbol (lib_id "Pale Slim Ghost:OLED_CH1117") (at 105.791 71.247 0) (unit 1)
-    (in_bom yes) (on_board yes) (dnp no) (fields_autoplaced)
+    (in_bom no) (on_board yes) (dnp no) (fields_autoplaced)
     (property "Reference" "U1" (at 116.84 71.755 0)
       (effects (font (size 1.27 1.27)) (justify left))
