File: eurorack/modules/pigeons/pigeons.kicad_sch (KiCad schematic)
At the start: 54 parts, among them J1 AudioJack3_SwitchTR, J10 AudioJack2_SwitchT, J11 AudioJack2_SwitchT, J12 AudioJack2_SwitchT, J13 Conn_02x05_Odd_Even, J14 Conn_01x04_Socket, J15 Conn_01x04_Pin, J2 AudioJack3_SwitchTR, J3 AudioJack3_SwitchTR, J4 AudioJack2_SwitchT, J5 AudioJack2_SwitchT, J6 AudioJack2_SwitchT, J7 AudioJack2_SwitchT, J8 AudioJack2_SwitchT, J9 AudioJack2_SwitchT, U1 TL074, U2 TL072

Commit message: jan 24
Connections:
- net +12V: now also U2.8 (V+); no longer U2.4 (V-)
- net -12V: now also U2.4 (V-); no longer U2.8 (V+)
Changed lines of the file:
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@@
     )
   )
-  (symbol (lib_id "Amplifier_Operational:TL072") (at 250.698 26.289 0) (mirror x) (unit 3)
+  (symbol (lib_id "Amplifier_Operational:TL072") (at 245.618 26.289 0) (mirror y) (unit 3)
     (in_bom yes) (on_board yes) (dnp no) (fields_autoplaced)
     (property "Reference" "U2" (at 248.92 25.654 0)
-      (effects (font (size 1.27 1.27)) (justify left))
+      (effects (font (size 1.27 1.27)) (justify right))
     )
     (property "Value" "TL072" (at 248.92 28.194 0)
-      (effects (font (size 1.27 1.27)) (justify left))
+      (effects (font (size 1.27 1.27)) (justify right))
     )
-    (property "Footprint" "Package_SO:SOIC-8_3.9x4.9mm_P1.27mm" (at 250.698 26.289 0)
+    (property "Footprint" "Package_SO:SOIC-8_3.9x4.9mm_P1.27mm" (at 245.618 26.289 0)
       (effects (font (size 1.27 1.27)) hide)
     )
-    (property "Datasheet" "http://www.ti.com/lit/ds/symlink/tl071.pdf" (at 250.698 26.289 0)
+    (property "Datasheet" "http://www.ti.com/lit/ds/symlink/tl071.pdf" (at 245.618 26.289 0)
       (effects (font (size 1.27 1.27)) hide)
     )
